File: Hardware/MICS-4514_CO_and_NOx_Sensor_Breakout.sch (EAGLE design)
At the start: 15 parts, among them Q2 MOSFET-NCHANNELBSS138

Commit message: Finished schematic. Added pre-heating FET.
Parts:
- removed LOGO2: SFE_LOGO_FLAME.1_INCH, SparkFun-Aesthetics:SFE_LOGO_FLAME.1_INCH
- removed LOGO3: SFE_LOGO_NAME_FLAME.1_INCH, SparkFun-Aesthetics:SFE_LOGO_NAME_FLAME.1_INCH
- removed U$1: MICS-4514, SparkFun-Sensors:MICS-4514
- added R4: 100k, SparkFun-Resistors:100KOHM1/10W1%(0603)
- added R5: 22K, SparkFun-Resistors:22KOHM1/10W1%(0603)
- added R6: 82, SparkFun-Resistors:RESISTOR0805-RES
- added R7: 47K, SparkFun-Resistors:47KOHM1/10W1%(0603)
- added U1: MICS-4514, SparkFun-Sensors:MICS-4514
- Q2: P_NAME (none) -> BSS138
- R1: device SparkFun-Resistors:RESISTOR0603 -> SparkFun-Resistors:RESISTOR0805-RES; DK_ID (none) -> 541-82.0CCT-ND; PROD_ID RES-12311 -> (none)
- R2: value 820 -> 51; PROD_ID RES-12313 -> RES-12314
- R3: value 51 -> 100; device SparkFun-Resistors:RESISTOR0603 -> SparkFun-Resistors:100OHM1/10W1%(0603); PROD_ID RES-12314 -> (none)
Connections:
- removed net VO: R2.2
- removed net VO_OX: JP2.2
- removed net VO_RED: JP2.3
- new net N$1: R1.2, U1.RH1_OX
- new net N$3: Q2.G, R3.2, R4.2
- new net N$6: Q2.D, R1.1, R2.2
- new net VNOX: JP2.2, R5.2, U1.RS1_OX
- new net VRED: JP2.3, R7.2, U1.RS1_RED
- net 5V: now also U1.RH2_OX, U1.RH2_RED, U1.RS2_OX, U1.RS2_RED
- net GND: now also Q2.S, R4.1, R5.1, R6.1, R7.1
- net N$2: now also R6.2, U1.RH1_RED; no longer R1.2
- net PRE: now also R3.1
Other:
- note added: "Shawn Hymel"
- note added: "v01"
- note removed: "N. Seidle Revision by Shawn Hymel"
- note removed: "v12"
- moved on the sheet: C1, JP2, Q2, R1, R2, R3

Commit message: Created initial layout.
Parts:
- renumbered JP2 to JP1
Changed lines of the file:
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@@
 <setting verticaltext="up"/>
 </settings>
-<grid distance="0.1" unitdist="inch" unit="inch" style="lines" multiple="1" display="yes" altdistance="0.01" altunitdist="inch" altunit="inch"/>
+<grid distance="0.1" unitdist="inch" unit="inch" style="lines" multiple="1" display="no" altdistance="0.01" altunitdist="inch" altunit="inch"/>
 <layers>
 <layer number="1" name="Top" color="4" fill="1" visible="no" active="no"/>
@@
 <attribute name="P_NAME" value="BSS138"/>
 </part>
-<part name="JP2" library="SparkFun-Connectors" deviceset="M05" device="LOCK"/>
+<part name="JP1" library="SparkFun-Connectors" deviceset="M05" device="LOCK"/>
 <part name="SUPPLY4" library="SparkFun-Aesthetics" deviceset="5V" device=""/>
 <part name="GND5" library="SparkFun-Aesthetics" deviceset="GND" device=""/>
@@
 <attribute name="P_NAME" x="109.22" y="96.52" size="1.778" layer="96"/>
 </instance>
-<instance part="JP2" gate="G$1" x="30.48" y="114.3" rot="MR180"/>
+<instance part="JP1" gate="G$1" x="30.48" y="114.3" rot="MR180"/>
 <instance part="SUPPLY4" gate="G$1" x="53.34" y="114.3"/>
 <instance part="GND5" gate="1" x="53.34" y="104.14"/>
@@
 </segment>
 <segment>
-<pinref part="JP2" gate="G$1" pin="4"/>
+<pinref part="JP1" gate="G$1" pin="4"/>
 <wire x1="38.1" y1="111.76" x2="53.34" y2="111.76" width="0.1524" layer="91"/>
 <wire x1="53.34" y1="111.76" x2="53.34" y2="114.3" width="0.1524" layer="91"/>
@@
 </segment>
 <segment>
-<pinref part="JP2" gate="G$1" pin="5"/>
+<pinref part="JP1" gate="G$1" pin="5"/>
 <wire x1="38.1" y1="109.22" x2="53.34" y2="109.22" width="0.1524" layer="91"/>
 <wire x1="53.34" y1="109.22" x2="53.34" y2="106.68" width="0.1524" layer="91"/>
@@
 </segment>
 <segment>
-<pinref part="JP2" gate="G$1" pin="2"/>
+<pinref part="JP1" gate="G$1" pin="2"/>
 <wire x1="38.1" y1="116.84" x2="40.64" y2="116.84" width="0.1524" layer="91"/>
 <label x="40.64" y="116.84" size="1.27" layer="95" xref="yes"/>
@@
 <net name="VRED" class="0">
 <segment>
-<pinref part="JP2" gate="G$1" pin="3"/>
+<pinref part="JP1" gate="G$1" pin="3"/>
 <wire x1="38.1" y1="114.3" x2="40.64" y2="114.3" width="0.1524" layer="91"/>
 <label x="40.64" y="114.3" size="1.27" layer="95" xref="yes"/>
@@
 <net name="PRE" class="0">
 <segment>
-<pinref part="JP2" gate="G$1" pin="1"/>
+<pinref part="JP1" gate="G$1" pin="1"/>
 <wire x1="38.1" y1="119.38" x2="40.64" y2="119.38" width="0.1524" layer="91"/>
 <label x="40.64" y="119.38" size="1.27" layer="95" xref="yes"/>
